Commit message: camera done

File: description/robot.urdf.xacro (robot description, xacro)
@@ -3,3 +3,6 @@
     <!-- Example link -->
     <xacro:include filename="robot_core.xacro" />
+    <xacro:include filename="gazebo_control.xacro"/>
+    <xacro:include filename="lidar.xacro"/>
+    <xacro:include filename="camera.xacro"/>
 </robot>

File: description/robot_core.xacro (robot description, xacro)
@@ -13,4 +13,7 @@
     <material name="black">
         <color rgba="0 0 0 1"/>
+    </material>
+    <material name="red">
+        <color rgba="1 0 0 1"/>
     </material>
  <!-- Base link -->
@@ -41,4 +44,7 @@
     </xacro:inertial_box>
 </link>
+<gazebo reference="chassis">
+        <material>Gazebo/White</material>
+</gazebo>
 <joint name="left_wheel_joint" type="continuous">
     <parent link="base_link"/>
@@ -64,4 +70,7 @@
     </xacro:inertial_cylinder>
 </link>
+<gazebo reference="left_wheel">
+        <material>Gazebo/Blue</material>
+</gazebo>
 <joint name="right_wheel_joint" type="continuous">
     <parent link="base_link"/>
@@ -87,4 +96,7 @@
     </xacro:inertial_cylinder>
 </link>
+<gazebo reference="right_wheel">
+        <material>Gazebo/Blue</material>
+</gazebo>
 <!-- CASTER WHEEL LINK -->
 <joint name="caster_wheel_joint" type="fixed">
@@ -109,3 +121,8 @@
     </xacro:inertial_sphere>
 </link>
+<gazebo reference="caster_wheel">
+        <material>Gazebo/Black</material>
+        <mu1 value="0.001"/>
+        <mu2 value="0.001"/>
+</gazebo>
 </robot>
